Commit message: Added RL Controller and added URDF

File: mbf_description/urdf/mbf.urdf (robot description, URDF)
Before this commit: robot mbf, 19 links, 18 joints
Links:
- link base_link: geometry 
- link chassis: mass 1.0 -> 2; geometry collision mesh filename=file://$(find mbf_description)/meshes/chassis.stl; visual mesh filename=file://$(find mbf_description)/meshes/chassis.stl
- link fl_feet_link: mass 0.035 -> 0.025; geometry collision mesh filename=file://$(find mbf_description)/meshes/feet.stl; visual mesh filename=file://$(find mbf_description)/meshes/feet.stl
- link fl_hip_link: mass 0.4 -> 0.6; geometry collision mesh filename=file://$(find mbf_description)/meshes/hip.stl; visual mesh filename=file://$(find mbf_description)/meshes/hip.stl
- link fl_knee_link: mass 0.035 -> 0.15; geometry collision mesh filename=file://$(find mbf_description)/meshes/knee.stl; visual mesh filename=file://$(find mbf_description)/meshes/knee.stl
- link fl_shoulder_link: geometry collision mesh filename=file://$(find mbf_description)/meshes/shoulder.stl; visual mesh filename=file://$(find mbf_description)/meshes/shoulder.stl
- link fr_feet_link: mass 0.035 -> 0.025; geometry collision mesh filename=file://$(find mbf_description)/meshes/feet.stl; visual mesh filename=file://$(find mbf_description)/meshes/feet.stl
- link fr_hip_link: mass 0.4 -> 0.6; geometry collision mesh filename=file://$(find mbf_description)/meshes/hip.stl; visual mesh filename=file://$(find mbf_description)/meshes/hip.stl
- link fr_knee_link: mass 0.035 -> 0.15; geometry collision mesh filename=file://$(find mbf_description)/meshes/knee.stl; visual mesh filename=file://$(find mbf_description)/meshes/knee.stl
- link fr_shoulder_link: geometry collision mesh filename=file://$(find mbf_description)/meshes/shoulder.stl; visual mesh filename=file://$(find mbf_description)/meshes/shoulder.stl
- link imu_link: mass 0.001 -> None; geometry 
- link rl_feet_link: mass 0.035 -> 0.025; geometry collision mesh filename=file://$(find mbf_description)/meshes/feet.stl; visual mesh filename=file://$(find mbf_description)/meshes/feet.stl
- link rl_hip_link: mass 0.4 -> 0.6; geometry collision mesh filename=file://$(find mbf_description)/meshes/hip.stl; visual mesh filename=file://$(find mbf_description)/meshes/hip.stl
- link rl_knee_link: mass 0.035 -> 0.15; geometry collision mesh filename=file://$(find mbf_description)/meshes/knee.stl; visual mesh filename=file://$(find mbf_description)/meshes/knee.stl
- link rl_shoulder_link: geometry collision mesh filename=file://$(find mbf_description)/meshes/shoulder.stl; visual mesh filename=file://$(find mbf_description)/meshes/shoulder.stl
- link rr_feet_link: mass 0.035 -> 0.025; geometry collision mesh filename=file://$(find mbf_description)/meshes/feet.stl; visual mesh filename=file://$(find mbf_description)/meshes/feet.stl
- link rr_hip_link: mass 0.4 -> 0.6; geometry collision mesh filename=file://$(find mbf_description)/meshes/hip.stl; visual mesh filename=file://$(find mbf_description)/meshes/hip.stl
- link rr_knee_link: mass 0.035 -> 0.15; geometry collision mesh filename=file://$(find mbf_description)/meshes/knee.stl; visual mesh filename=file://$(find mbf_description)/meshes/knee.stl
- link rr_shoulder_link: geometry collision mesh filename=file://$(find mbf_description)/meshes/shoulder.stl; visual mesh filename=file://$(find mbf_description)/meshes/shoulder.stl
Joints:
- removed joint floating_base
- added joint base_link_joint: type fixed, parent base_link, child chassis
- joint fl_feet_joint: axis (none) -> 0 0 1; limit (none) -> effort=10 velocity=10; origin xyz=0 0 -0.137 rpy=0 0 0 -> xyz=-0.000288395 -0 -0.148233 rpy=-0 -0 -0
- joint fl_hip_joint: limit lower=-1.5708 upper=1.5708 effort=10.0 velocity=10.0 -> lower=-2.5 upper=2.5 effort=10 velocity=10; origin xyz=0 0.085 0 rpy=0 0 0 -> xyz=0 0.081 -0 rpy=0 -0 -0
- joint fl_knee_joint: limit lower=-2.0944 upper=2.0944 effort=10.0 velocity=10.0 -> lower=-2.5 upper=0 effort=10 velocity=10
- joint fl_shoulder_joint: limit lower=-0.785398 upper=0.785398 effort=10.0 velocity=10.0 -> lower=-2.0 upper=2.0 effort=10 velocity=10; origin xyz=0.16 0.0425 0 rpy=0 0 0 -> xyz=0.1695 0.045 0 rpy=0 0 0
- joint fr_feet_joint: axis (none) -> 0 0 1; limit (none) -> effort=10 velocity=10; origin xyz=0 0 -0.137 rpy=0 0 0 -> xyz=-0.000288395 -0 -0.148233 rpy=-0 -0 -0
- joint fr_hip_joint: limit lower=-1.5708 upper=1.5708 effort=10.0 velocity=10.0 -> lower=-2.5 upper=2.5 effort=10 velocity=10; origin xyz=0 -0.085 0 rpy=0 0 0 -> xyz=0 -0.081 0 rpy=-0 -0 0
- joint fr_knee_joint: limit lower=-2.0944 upper=2.0944 effort=10.0 velocity=10.0 -> lower=-2.5 upper=0 effort=10 velocity=10; origin xyz=0 0 -0.12 rpy=0 0 0 -> xyz=0 0 -0.12 rpy=0 -0 -0
- joint fr_shoulder_joint: limit lower=-0.785398 upper=0.785398 effort=10.0 velocity=10.0 -> lower=-2.0 upper=2.0 effort=10 velocity=10; origin xyz=0.16 -0.0425 0 rpy=0 0 0 -> xyz=0.1695 -0.045 0 rpy=0 0 -0
- joint imu_joint: origin xyz=0 0 0 rpy=0 0 0 -> (none)
- joint rl_feet_joint: axis (none) -> 0 0 1; limit (none) -> effort=10 velocity=10; origin xyz=0 0 -0.137 rpy=0 0 0 -> xyz=-0.000288395 -0 -0.148233 rpy=-0 0 -0
- joint rl_hip_joint: limit lower=-1.5708 upper=1.5708 effort=10.0 velocity=10.0 -> lower=-2.5 upper=2.5 effort=10 velocity=10; origin xyz=0 0.085 0 rpy=0 0 0 -> xyz=0 0.081 -0 rpy=0 -0 0
- joint rl_knee_joint: limit lower=-2.0944 upper=2.0944 effort=10.0 velocity=10.0 -> lower=-2.5 upper=0 effort=10 velocity=10; origin xyz=0 0 -0.12 rpy=0 0 0 -> xyz=0 0 -0.12 rpy=0 -0 -0
- joint rl_shoulder_joint: limit lower=-0.785398 upper=0.785398 effort=10.0 velocity=10.0 -> lower=-2.0 upper=2.0 effort=10 velocity=10; origin xyz=-0.16 0.0425 0 rpy=0 0 0 -> xyz=-0.1695 0.045 0 rpy=0 -0 0
- joint rr_feet_joint: axis (none) -> 0 0 1; limit (none) -> effort=10 velocity=10; origin xyz=0 0 -0.137 rpy=0 0 0 -> xyz=-0.000288395 -0 -0.148233 rpy=-0 -0 -0
- joint rr_hip_joint: limit lower=-1.5708 upper=1.5708 effort=10.0 velocity=10.0 -> lower=-2.5 upper=2.5 effort=10 velocity=10; origin xyz=0 -0.085 0 rpy=0 0 0 -> xyz=0 -0.081 -0 rpy=0 -0 0
- joint rr_knee_joint: limit lower=-2.0944 upper=2.0944 effort=10.0 velocity=10.0 -> lower=-2.5 upper=0 effort=10 velocity=10; origin xyz=0 0 -0.12 rpy=0 0 0 -> xyz=0 0 -0.12 rpy=0 -0 0
- joint rr_shoulder_joint: limit lower=-0.785398 upper=0.785398 effort=10.0 velocity=10.0 -> lower=-2.0 upper=2.0 effort=10 velocity=10; origin xyz=-0.16 -0.0425 0 rpy=0 0 0 -> xyz=-0.1695 -0.045 0 rpy=0 -0 0

File: mbf_description/xacro/gazebo.xacro (robot description, xacro)
@@ -1,99 +1,71 @@
 <?xml version="1.0"?>
 <robot xmlns:xacro="http://www.ros.org/wiki/xacro">
-	<gazebo reference="imu_link">
-		<sensor name="imu_sensor" type="imu">
-			<plugin filename="libgazebo_ros_imu_sensor.so" name="imu_plugin">
-				<ros>
-					<namespace>/</namespace>
-					<remapping>~/out:=imu</remapping>
-				</ros>
-				<initial_orientation_as_reference>false</initial_orientation_as_reference>
-			</plugin>
-			<always_on>true</always_on>
-			<update_rate>100</update_rate>
-			<visualize>true</visualize>
-			<imu>
-				<angular_velocity>
-					<x>
-						<noise type="gaussian">
-							<mean>0.0</mean>
-							<stddev>2e-4</stddev>
-							<bias_mean>0.0000075</bias_mean>
-							<bias_stddev>0.0000008</bias_stddev>
-						</noise>
-					</x>
-					<y>
-						<noise type="gaussian">
-							<mean>0.0</mean>
-							<stddev>2e-4</stddev>
-							<bias_mean>0.0000075</bias_mean>
-							<bias_stddev>0.0000008</bias_stddev>
-						</noise>
-					</y>
-					<z>
-						<noise type="gaussian">
-							<mean>0.0</mean>
-							<stddev>2e-4</stddev>
-							<bias_mean>0.0000075</bias_mean>
-							<bias_stddev>0.0000008</bias_stddev>
-						</noise>
-					</z>
-				</angular_velocity>
-				<linear_acceleration>
-					<x>
-						<noise type="gaussian">
-							<mean>0.0</mean>
-							<stddev>1.7e-2</stddev>
-							<bias_mean>0.1</bias_mean>
-							<bias_stddev>0.001</bias_stddev>
-						</noise>
-					</x>
-					<y>
-						<noise type="gaussian">
-							<mean>0.0</mean>
-							<stddev>1.7e-2</stddev>
-							<bias_mean>0.1</bias_mean>
-							<bias_stddev>0.001</bias_stddev>
-						</noise>
-					</y>
-					<z>
-						<noise type="gaussian">
-							<mean>0.0</mean>
-							<stddev>1.7e-2</stddev>
-							<bias_mean>0.1</bias_mean>
-							<bias_stddev>0.001</bias_stddev>
-						</noise>
-					</z>
-				</linear_acceleration>
-			</imu>
-		</sensor>
-	</gazebo>
-	<gazebo reference="fl_feet_link">
-		<mu1>0.6</mu1>
-		<mu2>0.6</mu2>
-		<self_collide>1</self_collide>
-		<kp value="1000000.0"/>
-		<kd value="1.0"/>
-	</gazebo>
-	<gazebo reference="fr_feet_link">
-		<mu1>0.6</mu1>
-		<mu2>0.6</mu2>
-		<self_collide>1</self_collide>
-		<kp value="1000000.0"/>
-		<kd value="1.0"/>
-	</gazebo>
-	<gazebo reference="rl_feet_link">
-		<mu1>0.6</mu1>
-		<mu2>0.6</mu2>
-		<self_collide>1</self_collide>
-		<kp value="1000000.0"/>
-		<kd value="1.0"/>
-	</gazebo>
-	<gazebo reference="rr_feet_link">
-		<mu1>0.6</mu1>
-		<mu2>0.6</mu2>
-		<self_collide>1</self_collide>
-		<kp value="1000000.0"/>
-		<kd value="1.0"/>
-	</gazebo>
+    <gazebo reference="imu_link">
+        <sensor name="imu_sensor" type="imu">
+            <plugin filename="libgazebo_ros_imu_sensor.so" name="imu_plugin">
+                <ros>
+                    <namespace>/</namespace>
+                    <remapping>~/out:=imu</remapping>
+                </ros>
+                <initial_orientation_as_reference>false</initial_orientation_as_reference>
+            </plugin>
+            <always_on>true</always_on>
+            <update_rate>100</update_rate>
+            <visualize>true</visualize>
+            <imu>
+                <angular_velocity>
+                    <x>
+                        <noise type="gaussian">
+                            <mean>0.0</mean>
+                            <stddev>2e-4</stddev>
+                            <bias_mean>0.0000075</bias_mean>
+                            <bias_stddev>0.0000008</bias_stddev>
+                        </noise>
+                    </x>
+                    <y>
+                        <noise type="gaussian">
+                            <mean>0.0</mean>
+                            <stddev>2e-4</stddev>
+                            <bias_mean>0.0000075</bias_mean>
+                            <bias_stddev>0.0000008</bias_stddev>
+                        </noise>
+                    </y>
+                    <z>
+                        <noise type="gaussian">
+                            <mean>0.0</mean>
+                            <stddev>2e-4</stddev>
+                            <bias_mean>0.0000075</bias_mean>
+                            <bias_stddev>0.0000008</bias_stddev>
+                        </noise>
+                    </z>
+                </angular_velocity>
+                <linear_acceleration>
+                    <x>
+                        <noise type="gaussian">
+                            <mean>0.0</mean>
+                            <stddev>1.7e-2</stddev>
+                            <bias_mean>0.1</bias_mean>
+                            <bias_stddev>0.001</bias_stddev>
+                        </noise>
+                    </x>
+                    <y>
+                        <noise type="gaussian">
+                            <mean>0.0</mean>
+                            <stddev>1.7e-2</stddev>
+                            <bias_mean>0.1</bias_mean>
+                            <bias_stddev>0.001</bias_stddev>
+                        </noise>
+                    </y>
+                    <z>
+                        <noise type="gaussian">
+                            <mean>0.0</mean>
+                            <stddev>1.7e-2</stddev>
+                            <bias_mean>0.1</bias_mean>
+                            <bias_stddev>0.001</bias_stddev>
+                        </noise>
+                    </z>
+                </linear_acceleration>
+            </imu>
+        </sensor>
+    </gazebo>
 </robot>

File: mbf_description/xacro/robot.xacro (robot description, xacro)
@@ -1,69 +1,9 @@
 <?xml version="1.0"?>
-<robot name="mbf"
-    xmlns:xacro="http://www.ros.org/wiki/xacro">
-    <xacro:include filename="$(find mbf_description)/xacro/const.xacro"/>
-    <!-- <xacro:include filename="$(find mbf_description)/xacro/materials.xacro"/> -->
-    <xacro:include filename="$(find mbf_description)/xacro/leg.xacro"/>
-    <link name="base_link">
-        <visual>
-            <origin rpy="0 0 0" xyz="0 0 0"/>
-            <geometry>
-                <box size="0.001 0.001 0.001"/>
-            </geometry>
-        </visual>
-    </link>
-    <joint name="floating_base" type="fixed">
-        <origin rpy="0 0 0" xyz="0 0 0"/>
-        <parent link="base_link"/>
-        <child link="chassis"/>
-    </joint>
-    <link name="chassis">
-        <visual>
-            <origin rpy="0 0 0" xyz="0 0 0"/>
-            <geometry>
-                <mesh filename="file://$(find mbf_description)/meshes/Chassis.stl" scale="0.001 0.001 0.001"/>
-            </geometry>
-            <!-- <material name="grey"/> -->
-        </visual>
-        <collision>
-            <origin rpy="0 0 0" xyz="0 0 0"/>
-            <geometry>
-                <box size="${chassis_length} ${chassis_width} ${chassis_height}"/>
-            </geometry>
-        </collision>
-        <inertial>
-            <origin xyz="0 0 0" />
-            <mass value="${chassis_mass}" />
-            <inertia ixx="${(1/12) * chassis_mass * (chassis_width * chassis_width + chassis_height * chassis_height)}" ixy="0.0" ixz="0.0" iyy="${(1/12) * chassis_mass * (chassis_length * chassis_length + chassis_height * chassis_height)}" iyz="0.0" izz="${(1/12) * chassis_mass * (chassis_length * chassis_length + chassis_width * chassis_width)}" />
-        </inertial>
-    </link>
-    <joint name="imu_joint" type="fixed">
-        <parent link="chassis"/>
-        <child link="imu_link"/>
-        <origin rpy="0 0 0" xyz="0 0 0"/>
-    </joint>
-    <link name="imu_link">
-        <inertial>
-            <mass value="0.001"/>
-            <origin rpy="0 0 0" xyz="0 0 0"/>
-            <inertia ixx="0.0001" ixy="0" ixz="0" iyy="0.0001" iyz="0" izz="0.0001"/>
-        </inertial>
-        <visual>
-            <origin rpy="0 0 0" xyz="0 0 0"/>
-            <geometry>
-                <box size="0.001 0.001 0.001"/>
-            </geometry>
-            <!-- <material name="red"/> -->
-        </visual>
-        <collision>
-            <origin rpy="0 0 0" xyz="0 0 0"/>
-            <geometry>
-                <box size=".001 .001 .001"/>
-            </geometry>
-        </collision>
-    </link>
-    <xacro:leg leg="fl"/>
-    <xacro:leg leg="fr"/>
-    <xacro:leg leg="rl"/>
-    <xacro:leg leg="rr"/>
+<robot xmlns:xacro="http://www.ros.org/wiki/xacro" name="robot">
+    <xacro:arg name="use_sim" default="false"/>
+    <xacro:include filename="$(find mbf_description)/urdf/mbf.urdf"/>
+    <xacro:include filename="$(find mbf_description)/ros2_control/ros2_control.xacro"/>
+    <xacro:if value="$(arg use_sim)">
+        <xacro:include filename="$(find mbf_description)/xacro/gazebo.xacro"/>
+    </xacro:if>
 </robot>

Commit message: Add minimal readme and modified little modifications

File: mbf_description/urdf/mbf.urdf (robot description, URDF)
Before this commit: robot mbf, 19 links, 18 joints
Joints:
- joint fl_hip_joint: limit lower=-2.5 upper=2.5 effort=10 velocity=10 -> lower=-1.5708 upper=3.5 effort=10 velocity=10
- joint fl_shoulder_joint: limit lower=-2.0 upper=2.0 effort=10 velocity=10 -> lower=-1.0472 upper=1.0472 effort=10 velocity=10
- joint fr_hip_joint: limit lower=-2.5 upper=2.5 effort=10 velocity=10 -> lower=-1.5708 upper=3.5 effort=10 velocity=10
- joint fr_shoulder_joint: limit lower=-2.0 upper=2.0 effort=10 velocity=10 -> lower=-1.0472 upper=1.0472 effort=10 velocity=10
- joint rl_hip_joint: limit lower=-2.5 upper=2.5 effort=10 velocity=10 -> lower=-1.5708 upper=3.5 effort=10 velocity=10
- joint rl_shoulder_joint: limit lower=-2.0 upper=2.0 effort=10 velocity=10 -> lower=-1.0472 upper=1.0472 effort=10 velocity=10
- joint rr_hip_joint: limit lower=-2.5 upper=2.5 effort=10 velocity=10 -> lower=-1.5708 upper=3.5 effort=10 velocity=10
- joint rr_shoulder_joint: limit lower=-2.0 upper=2.0 effort=10 velocity=10 -> lower=-1.0472 upper=1.0472 effort=10 velocity=10

Commit message: Updated robot model and added EE policy

File: mbf_description/urdf/mbf.urdf (robot description, URDF)
Before this commit: robot mbf, 19 links, 18 joints
Links:
- link chassis: mass 2 -> 2.0
Joints:
- joint fl_shoulder_joint: origin xyz=0.1695 0.045 0 rpy=0 0 0 -> xyz=0.1805 0.045 -0 rpy=-0 0 0
- joint fr_shoulder_joint: origin xyz=0.1695 -0.045 0 rpy=0 0 -0 -> xyz=0.1805 -0.045 -0 rpy=0 0 0
- joint rl_feet_joint: origin xyz=-0.000288395 -0 -0.148233 rpy=-0 0 -0 -> xyz=-0.000288395 -0 -0.148233 rpy=-0 -0 -0
- joint rl_shoulder_joint: origin xyz=-0.1695 0.045 0 rpy=0 -0 0 -> xyz=-0.1805 0.045 0 rpy=-0 0 -0
- joint rr_feet_joint: origin xyz=-0.000288395 -0 -0.148233 rpy=-0 -0 -0 -> xyz=-0.000288395 -0 -0.148233 rpy=0 0 -0
- joint rr_shoulder_joint: origin xyz=-0.1695 -0.045 0 rpy=0 -0 0 -> xyz=-0.1805 -0.045 0 rpy=-0 0 0
