Commit message: Tuned for FR leg, but need to fix hardware interface manual offset

File: mbf_description/ros2_control/ros2_control.xacro (robot description, xacro)
@@ -8,5 +8,5 @@
                 <param name="can">can0</param>
             </hardware>
-            <joint name="fl_shoulder_joint">
+            <!-- <joint name="fl_shoulder_joint">
                 <param name="node_id">0</param>
                 <param name="reduction_ratio">8.0</param>
@@ -28,11 +28,11 @@
                 <param name="offset">0.0</param>
                 <param name="axis_direction">1.0</param>
-            </joint>
+            </joint> -->
             <joint name="fr_shoulder_joint">
                 <param name="node_id">3</param>
                 <param name="reduction_ratio">8.0</param>
                 <param name="auto_offset">1</param>
-                <param name="offset">0.0</param>
-                <param name="axis_direction">1.0</param>
+                <param name="offset">0.524</param>
+                <param name="axis_direction">-1</param>
             </joint>
             <joint name="fr_hip_joint">
@@ -40,5 +40,5 @@
                 <param name="reduction_ratio">8.0</param>
                 <param name="auto_offset">1</param>
-                <param name="offset">0.0</param>
+                <param name="offset">3.142</param>
                 <param name="axis_direction">1.0</param>
             </joint>
@@ -47,8 +47,8 @@
                 <param name="reduction_ratio">8.0</param>
                 <param name="auto_offset">1</param>
-                <param name="offset">0.0</param>
-                <param name="axis_direction">1.0</param>
-            </joint>
-            <joint name="rl_shoulder_joint">
+                <param name="offset">2.5</param>
+                <param name="axis_direction">1.0</param>
+            </joint>
+            <!-- <joint name="rl_shoulder_joint">
                 <param name="node_id">6</param>
                 <param name="reduction_ratio">8.0</param>
@@ -91,5 +91,5 @@
                 <param name="offset">0.0</param>
                 <param name="axis_direction">1.0</param>
-            </joint>
+            </joint> -->
         </ros2_control>
     </xacro:unless>

Commit message: Updated robot_hardware interface, can_service, and urdf. Tuned defaults for joints as well

File: mbf_description/ros2_control/ros2_control.xacro (robot description, xacro)
@@ -9,12 +9,12 @@
                 <param name="can">can0</param>
             </hardware>
-            <!-- <joint name="fl_shoulder_joint">
+            <joint name="fl_shoulder_joint">
                 <param name="node_id">0</param>
                 <param name="reduction_ratio">8.0</param>
                 <param name="auto_offset">1</param>
-                <param name="offset">0.0</param>
-                <param name="axis_direction">1.0</param>
-            </joint>
-            <joint name="fl_hip_joint">
+                <param name="offset">0.4</param>
+                <param name="axis_direction">-1.0</param>
+            </joint>
+            <!-- <joint name="fl_hip_joint">
                 <param name="node_id">1</param>
                 <param name="reduction_ratio">8.0</param>
@@ -34,8 +34,8 @@
                 <param name="reduction_ratio">8.0</param>
                 <param name="auto_offset">1</param>
-                <param name="offset">-0.26</param>
+                <param name="offset">-0.4</param>
                 <param name="axis_direction">-1</param>
             </joint>
-            <joint name="fr_hip_joint">
+            <!-- <joint name="fr_hip_joint">
                 <param name="node_id">4</param>
                 <param name="reduction_ratio">8.0</param>
@@ -43,6 +43,6 @@
                 <param name="offset">-3.14</param>
                 <param name="axis_direction">1</param>
-            </joint>
-            <joint name="fr_knee_joint">
+            </joint> -->
+            <!-- <joint name="fr_knee_joint">
                 <param name="node_id">5</param>
                 <param name="reduction_ratio">8.0</param>
@@ -50,5 +50,5 @@
                 <param name="offset">2.5</param>
                 <param name="axis_direction">1</param>
-            </joint>
+            </joint> -->
             <!-- <joint name="rl_shoulder_joint">
                 <param name="node_id">6</param>

File: mbf_description/urdf/mbf.urdf (robot description, URDF)
Before this commit: robot mbf, 19 links, 18 joints
Links:
- removed link imu_link
- added link base_imu_link
Joints:
- joint imu_joint: child imu_link -> base_imu_link

Commit message: Tuned defaults for front legs

File: mbf_description/ros2_control/ros2_control.xacro (robot description, xacro)
@@ -5,5 +5,5 @@
             <hardware>
                 <plugin>robot_ros2_control/RobotHardwareInterface</plugin>
-                <param name="logging">1</param>
+                <param name="logging">0</param>
                 <param name="read_torques">0</param>
                 <param name="can">can0</param>
@@ -16,10 +16,10 @@
                 <param name="axis_direction">-1.0</param>
             </joint>
-            <!-- <joint name="fl_hip_joint">
+            <joint name="fl_hip_joint">
                 <param name="node_id">1</param>
                 <param name="reduction_ratio">8.0</param>
                 <param name="auto_offset">1</param>
-                <param name="offset">0.0</param>
-                <param name="axis_direction">1.0</param>
+                <param name="offset">1.57</param>
+                <param name="axis_direction">-1.0</param>
             </joint>
             <joint name="fl_knee_joint">
@@ -27,7 +27,7 @@
                 <param name="reduction_ratio">8.0</param>
                 <param name="auto_offset">1</param>
-                <param name="offset">0.0</param>
-                <param name="axis_direction">1.0</param>
-            </joint> -->
+                <param name="offset">2.5</param>
+                <param name="axis_direction">-1.0</param>
+            </joint>
             <joint name="fr_shoulder_joint">
                 <param name="node_id">3</param>
@@ -37,12 +37,12 @@
                 <param name="axis_direction">-1</param>
             </joint>
-            <!-- <joint name="fr_hip_joint">
+            <joint name="fr_hip_joint">
                 <param name="node_id">4</param>
                 <param name="reduction_ratio">8.0</param>
                 <param name="auto_offset">1</param>
-                <param name="offset">-3.14</param>
+                <param name="offset">1.57</param>
                 <param name="axis_direction">1</param>
-            </joint> -->
-            <!-- <joint name="fr_knee_joint">
+            </joint>
+            <joint name="fr_knee_joint">
                 <param name="node_id">5</param>
                 <param name="reduction_ratio">8.0</param>
@@ -50,5 +50,5 @@
                 <param name="offset">2.5</param>
                 <param name="axis_direction">1</param>
-            </joint> -->
+            </joint>
             <!-- <joint name="rl_shoulder_joint">
                 <param name="node_id">6</param>

Commit message: Tuned all odrive offsets, still need reworking on improving ros2 control rate

File: mbf_description/ros2_control/ros2_control.xacro (robot description, xacro)
@@ -13,5 +13,5 @@
                 <param name="reduction_ratio">8.0</param>
                 <param name="auto_offset">1</param>
-                <param name="offset">0.4</param>
+                <param name="offset">-0.4</param>
                 <param name="axis_direction">-1.0</param>
             </joint>
@@ -20,5 +20,5 @@
                 <param name="reduction_ratio">8.0</param>
                 <param name="auto_offset">1</param>
-                <param name="offset">1.57</param>
+                <param name="offset">-1.5708</param>
                 <param name="axis_direction">-1.0</param>
             </joint>
@@ -34,5 +34,5 @@
                 <param name="reduction_ratio">8.0</param>
                 <param name="auto_offset">1</param>
-                <param name="offset">-0.4</param>
+                <param name="offset">0.4</param>
                 <param name="axis_direction">-1</param>
             </joint>
@@ -41,5 +41,5 @@
                 <param name="reduction_ratio">8.0</param>
                 <param name="auto_offset">1</param>
-                <param name="offset">1.57</param>
+                <param name="offset">-1.5708</param>
                 <param name="axis_direction">1</param>
             </joint>
@@ -51,9 +51,9 @@
                 <param name="axis_direction">1</param>
             </joint>
-            <!-- <joint name="rl_shoulder_joint">
+            <joint name="rl_shoulder_joint">
                 <param name="node_id">6</param>
                 <param name="reduction_ratio">8.0</param>
                 <param name="auto_offset">1</param>
-                <param name="offset">0.0</param>
+                <param name="offset">-0.4</param>
                 <param name="axis_direction">1.0</param>
             </joint>
@@ -62,6 +62,6 @@
                 <param name="reduction_ratio">8.0</param>
                 <param name="auto_offset">1</param>
-                <param name="offset">0.0</param>
-                <param name="axis_direction">1.0</param>
+                <param name="offset">-1.5708</param>
+                <param name="axis_direction">-1.0</param>
             </joint>
             <joint name="rl_knee_joint">
@@ -69,6 +69,6 @@
                 <param name="reduction_ratio">8.0</param>
                 <param name="auto_offset">1</param>
-                <param name="offset">0.0</param>
-                <param name="axis_direction">1.0</param>
+                <param name="offset">2.5</param>
+                <param name="axis_direction">-1.0</param>
             </joint>
             <joint name="rr_shoulder_joint">
@@ -76,5 +76,5 @@
                 <param name="reduction_ratio">8.0</param>
                 <param name="auto_offset">1</param>
-                <param name="offset">0.0</param>
+                <param name="offset">0.4</param>
                 <param name="axis_direction">1.0</param>
             </joint>
@@ -83,5 +83,5 @@
                 <param name="reduction_ratio">8.0</param>
                 <param name="auto_offset">1</param>
-                <param name="offset">0.0</param>
+                <param name="offset">-1.5708</param>
                 <param name="axis_direction">1.0</param>
             </joint>
@@ -90,7 +90,7 @@
                 <param name="reduction_ratio">8.0</param>
                 <param name="auto_offset">1</param>
-                <param name="offset">0.0</param>
-                <param name="axis_direction">1.0</param>
-            </joint> -->
+                <param name="offset">2.5</param>
+                <param name="axis_direction">1.0</param>
+            </joint>
         </ros2_control>
     </xacro:unless>
